File: _saved_nixie_tube.sch (KiCad schematic (older format))
At the start: 18 parts, among them J11 dc003a, Q1 SS8550, Q2 FQD5N60C, U1 MC34063

Commit message: finalize position of component
Parts:
- added Q3: Q_NPN_BCE, TO_SOT_Packages_SMD:SOT-23, symbol Q_NPN_BCE
- added Q4: Q_PMOS_GDS, nixie-tube-fp:TO-252-2-ds, symbol Q_PMOS_GDS
- added R4, R5: R, Resistors_SMD:R_0603, symbol R
- C1, C3, C4: footprint Capacitors_SMD:C_0603_HandSoldering -> Capacitors_SMD:C_0603
- J1: renamed from J?; footprint (none) -> Pin_Headers:Pin_Header_Angled_1x05_Pitch2.54mm
- J2: renamed from J?; footprint (none) -> Socket_Strips:Socket_Strip_Angled_1x05_Pitch2.54mm
- J3: renamed from J?; footprint (none) -> Pin_Headers:Pin_Header_Angled_1x01_Pitch2.54mm
- J4: renamed from J?; footprint (none) -> Socket_Strips:Socket_Strip_Angled_1x01_Pitch2.54mm
- R1, R2, R3: footprint Resistors_SMD:R_0603_HandSoldering -> Resistors_SMD:R_0603
Connections:
- wire segments 46 -> 51
Changed lines of the file:
@@
 F 0 "R2" V 5630 3200 50  0000 C CNN
 F 1 "470K" V 5550 3200 50  0000 C CNN
-F 2 "Resistors_SMD:R_0603_HandSoldering" V 5480 3200 50  0001 C CNN
+F 2 "Resistors_SMD:R_0603" V 5480 3200 50  0001 C CNN
 F 3 "" H 5550 3200 50  0000 C CNN
 	1    5550 3200
@@
 F 0 "R3" V 5630 3750 50  0000 C CNN
 F 1 "3K" V 5550 3750 50  0000 C CNN
-F 2 "Resistors_SMD:R_0603_HandSoldering" V 5480 3750 50  0001 C CNN
+F 2 "Resistors_SMD:R_0603" V 5480 3750 50  0001 C CNN
 F 3 "" H 5550 3750 50  0000 C CNN
 	1    5550 3750
@@
 F 0 "C3" H 5325 3900 50  0000 L CNN
 F 1 "0.01uF" H 5325 3700 50  0000 L CNN
-F 2 "Capacitors_SMD:C_0603_HandSoldering" H 5338 3650 50  0001 C CNN
+F 2 "Capacitors_SMD:C_0603" H 5338 3650 50  0001 C CNN
 F 3 "" H 5300 3800 50  0000 C CNN
 	1    5300 3800
@@
 F 0 "R1" V 4030 3550 50  0000 C CNN
 F 1 "1k0" V 3950 3550 50  0000 C CNN
-F 2 "Resistors_SMD:R_0603_HandSoldering" V 3880 3550 50  0001 C CNN
+F 2 "Resistors_SMD:R_0603" V 3880 3550 50  0001 C CNN
 F 3 "" H 3950 3550 50  0000 C CNN
 	1    3950 3550
@@
 F 0 "C1" H 3075 3550 50  0000 L CNN
 F 1 "20nF" H 3075 3350 50  0000 L CNN
-F 2 "Capacitors_SMD:C_0603_HandSoldering" H 3088 3300 50  0001 C CNN
+F 2 "Capacitors_SMD:C_0603" H 3088 3300 50  0001 C CNN
 F 3 "" H 3050 3450 50  0000 C CNN
 	1    3050 3450
@@
 F 0 "C4" H 5975 3050 50  0000 L CNN
 F 1 "2.2uF" H 6000 2750 50  0000 L CNN
-F 2 "Capacitors_SMD:C_0603_HandSoldering" H 5988 2800 50  0001 C CNN
+F 2 "Capacitors_SMD:C_0603" H 5988 2800 50  0001 C CNN
 F 3 "" H 5950 2950 50  0000 C CNN
 F 4 "250V" H 6100 2850 60  0000 C CNN "voltage"
@@
 1.25V
 $Comp
-L GND #PWR08
+L GND #PWR07
 U 1 1 59D52828
 P 3050 3600
-F 0 "#PWR08" H 3050 3350 50  0001 C CNN
+F 0 "#PWR07" H 3050 3350 50  0001 C CNN
 F 1 "GND" H 3050 3450 50  0000 C CNN
 F 2 "" H 3050 3600 50  0000 C CNN
@@
 +180V
 $Comp
-L GND #PWR09
+L GND #PWR08
 U 1 1 59D52C94
 P 3950 3700
-F 0 "#PWR09" H 3950 3450 50  0001 C CNN
+F 0 "#PWR08" H 3950 3450 50  0001 C CNN
 F 1 "GND" H 3950 3550 50  0000 C CNN
 F 2 "" H 3950 3700 50  0000 C CNN
@@
 $EndComp
 $Comp
-L GND #PWR010
+L GND #PWR09
 U 1 1 59D52CCD
 P 4300 3700
-F 0 "#PWR010" H 4300 3450 50  0001 C CNN
+F 0 "#PWR09" H 4300 3450 50  0001 C CNN
 F 1 "GND" H 4300 3550 50  0000 C CNN
 F 2 "" H 4300 3700 50  0000 C CNN
@@
 $EndComp
 $Comp
-L GND #PWR011
+L GND #PWR010
 U 1 1 59D51046
 P 2450 3925
-F 0 "#PWR011" H 2450 3675 50  0001 C CNN
+F 0 "#PWR010" H 2450 3675 50  0001 C CNN
 F 1 "GND" H 2450 3775 50  0000 C CNN
 F 2 "" H 2450 3925 50  0000 C CNN
@@
 $EndComp
 $Comp
-L Conn_01x01_Female J?
+L Conn_01x01_Female J4
 U 1 1 59E5D8C8
 P 7500 2325
-F 0 "J?" H 7500 2425 50  0000 C CNN
+F 0 "J4" H 7500 2425 50  0000 C CNN
 F 1 "Conn_01x01_Female" H 7500 2225 50  0000 C CNN
-F 2 "" H 7500 2325 50  0001 C CNN
+F 2 "Socket_Strips:Socket_Strip_Angled_1x01_Pitch2.54mm" H 7500 2325 50  0001 C CNN
 F 3 "" H 7500 2325 50  0001 C CNN
 	1    7500 2325
@@
 $EndComp
 $Comp
-L Conn_01x01_Male J?
+L Conn_01x01_Male J3
 U 1 1 59E5D935
 P 6550 2325
-F 0 "J?" H 6550 2425 50  0000 C CNN
+F 0 "J3" H 6550 2425 50  0000 C CNN
 F 1 "Conn_01x01_Male" H 6550 2225 50  0000 C CNN
-F 2 "" H 6550 2325 50  0001 C CNN
+F 2 "Pin_Headers:Pin_Header_Angled_1x01_Pitch2.54mm" H 6550 2325 50  0001 C CNN
 F 3 "" H 6550 2325 50  0001 C CNN
 	1    6550 2325
@@
 $EndComp
 $Comp
-L Conn_01x05_Female J?
+L Conn_01x05_Female J2
 U 1 1 59E5DA12
 P 3275 4900
-F 0 "J?" H 3275 5200 50  0000 C CNN
+F 0 "J2" H 3275 5200 50  0000 C CNN
 F 1 "Conn_01x05_Female" H 3275 4600 50  0000 C CNN
-F 2 "" H 3275 4900 50  0001 C CNN
+F 2 "Socket_Strips:Socket_Strip_Angled_1x05_Pitch2.54mm" H 3275 4900 50  0001 C CNN
 F 3 "" H 3275 4900 50  0001 C CNN
 	1    3275 4900
@@
 $EndComp
 $Comp
-L Conn_01x05_Male J?
+L Conn_01x05_Male J1
 U 1 1 59E5DABD
 P 2000 4900
-F 0 "J?" H 2000 5200 50  0000 C CNN
+F 0 "J1" H 2000 5200 50  0000 C CNN
 F 1 "Conn_01x05_Male" H 2000 4600 50  0000 C CNN
-F 2 "" H 2000 4900 50  0001 C CNN
+F 2 "Pin_Headers:Pin_Header_Angled_1x05_Pitch2.54mm" H 2000 4900 50  0001 C CNN
 F 3 "" H 2000 4900 50  0001 C CNN
 	1    2000 4900
@@
 MOSi
 $Comp
-L +9V #PWR?
+L +9V #PWR011
 U 1 1 59E5E8EF
 P 2250 3700
-F 0 "#PWR?" H 2250 3550 50  0001 C CNN
+F 0 "#PWR011" H 2250 3550 50  0001 C CNN
 F 1 "+9V" H 2250 3840 50  0000 C CNN
 F 2 "" H 2250 3700 50  0001 C CNN
@@
 Connection ~ 2400 3925
 Wire Wire Line
-	2025 2200 4800 2200
-Wire Wire Line
 	2200 4700 3075 4700
 Wire Wire Line
@@
 	2200 5100 3075 5100
 Wire Wire Line
-	2025 3775 2250 3775
-Wire Wire Line
 	2250 3775 2250 3700
 $Comp
-L +9V #PWR?
-U 1 1 59E5EBB2
-P 2025 2200
-F 0 "#PWR?" H 2025 2050 50  0001 C CNN
-F 1 "+9V" H 2025 2340 50  0000 C CNN
-F 2 "" H 2025 2200 50  0001 C CNN
-F 3 "" H 2025 2200 50  0001 C CNN
-	1    2025 2200
-	1    0    0    -1
-$EndComp
-$Comp
-L +9V #PWR?
+L +9V #PWR012
 U 1 1 59E5EF02
 P 2675 4500
-F 0 "#PWR?" H 2675 4350 50  0001 C CNN
+F 0 "#PWR012" H 2675 4350 50  0001 C CNN
 F 1 "+9V" H 2675 4640 50  0000 C CNN
 F 2 "" H 2675 4500 50  0001 C CNN
@@
 Connection ~ 2675 4700
 $Comp
-L GND #PWR?
+L GND #PWR013
 U 1 1 59E5EFC2
 P 2900 4600
-F 0 "#PWR?" H 2900 4350 50  0001 C CNN
+F 0 "#PWR013" H 2900 4350 50  0001 C CNN
 F 1 "GND" H 2900 4450 50  0000 C CNN
 F 2 "" H 2900 4600 50  0001 C CNN
@@
 Text Notes 6800 2275 0    60   ~ 0
 +180V
+Wire Wire Line
+	2025 2200 4800 2200
+$Comp
+L +9V #PWR014
+U 1 1 59E606F5
+P 1200 2200
+F 0 "#PWR014" H 1200 2050 50  0001 C CNN
+F 1 "+9V" H 1200 2340 50  0000 C CNN
+F 2 "" H 1200 2200 50  0001 C CNN
+F 3 "" H 1200 2200 50  0001 C CNN
+	1    1200 2200
+	1    0    0    -1
+$EndComp
+Wire Wire Line
+	2250 3775 1825 3775
+$Comp
+L R R5
+U 1 1 59E60FCF
+P 1400 2475
+F 0 "R5" V 1480 2475 50  0000 C CNN
+F 1 "R" V 1400 2475 50  0000 C CNN
+F 2 "Resistors_SMD:R_0603" V 1330 2475 50  0001 C CNN
+F 3 "" H 1400 2475 50  0001 C CNN
+	1    1400 2475
+	1    0    0    -1
+$EndComp
+$Comp
+L Q_NPN_BCE Q3
+U 1 1 59E61059
+P 1725 2900
+F 0 "Q3" H 1925 2950 50  0000 L CNN
+F 1 "Q_NPN_BCE" H 1925 2850 50  0000 L CNN
+F 2 "TO_SOT_Packages_SMD:SOT-23" H 1925 3000 50  0001 C CNN
+F 3 "" H 1725 2900 50  0001 C CNN
+	1    1725 2900
+	1    0    0    -1
+$EndComp
+Wire Wire Line
+	1200 2200 1625 2200
+Wire Wire Line
+	1400 2325 1400 2200
+Connection ~ 1400 2200
+Wire Wire Line
+	1400 2625 1400 2700
+Wire Wire Line
+	1400 2700 1825 2700
+Wire Wire Line
+	1825 2700 1825 2500
+$Comp
+L R R4
+U 1 1 59E6131F
+P 1375 2900
+F 0 "R4" V 1455 2900 50  0000 C CNN
+F 1 "R" V 1375 2900 50  0000 C CNN
+F 2 "Resistors_SMD:R_0603" V 1305 2900 50  0001 C CNN
+F 3 "" H 1375 2900 50  0001 C CNN
+	1    1375 2900
+	0    1    1    0
+$EndComp
+Text Label 1225 2900 2    60   ~ 0
+PWREN
+$Comp
+L GND #PWR015
+U 1 1 59E613BB
+P 1825 3100
+F 0 "#PWR015" H 1825 2850 50  0001 C CNN
+F 1 "GND" H 1825 2950 50  0000 C CNN
+F 2 "" H 1825 3100 50  0001 C CNN
+F 3 "" H 1825 3100 50  0001 C CNN
+	1    1825 3100
+	1    0    0    -1
+$EndComp
+$Comp
+L Q_PMOS_GDS Q4
+U 1 1 59E61F36
+P 1825 2300
+F 0 "Q4" H 2025 2350 50  0000 L CNN
+F 1 "Q_PMOS_GDS" H 2025 2250 50  0000 L CNN
+F 2 "nixie-tube-fp:TO-252-2-ds" H 2025 2400 50  0001 C CNN
+F 3 "" H 1825 2300 50  0001 C CNN
+	1    1825 2300
+	0    1    -1   0
+$EndComp
 $EndSCHEMATC
