File: nixie_tube.sch (KiCad schematic (older format))
At the start: 18 parts, among them J1 Conn_01x05_Male, J11 dc003a, J2 Conn_01x05_Female, J3 Conn_01x01_Male, J4 Conn_01x01_Female, Q1 SS8550, Q2 FQD5N60C, U1 MC34063

Commit message: rearrange components
Parts:
- added Q3: Q_NPN_BCE, TO_SOT_Packages_SMD:SOT-23, symbol Q_NPN_BCE
- added Q4: Q_PMOS_GDS, nixie-tube-fp:TO-252-2-ds, symbol Q_PMOS_GDS
- added R4, R5: R, Resistors_SMD:R_0603, symbol R
Connections:
- net +9V: now also Q4.3 (S), R5.1; no longer C2.1, L1.1, U1.1, U1.6 (V+), U1.7 (Isc), U1.8 (C0)
- net GND: now also Q3.3 (E)
- net PWREN: now also R4.2
- new net: C2.1, L1.1, Q4.2 (D), U1.1, U1.6 (V+), U1.7 (Isc), U1.8 (C0)
- new net: Q3.2 (C), Q4.1 (G), R5.2
- new net: Q3.1 (B), R4.1
Changed lines of the file:
@@
 L +9V #PWR014
 U 1 1 59E606F5
-P 2025 2200
-F 0 "#PWR014" H 2025 2050 50  0001 C CNN
-F 1 "+9V" H 2025 2340 50  0000 C CNN
-F 2 "" H 2025 2200 50  0001 C CNN
-F 3 "" H 2025 2200 50  0001 C CNN
-	1    2025 2200
+P 1200 2200
+F 0 "#PWR014" H 1200 2050 50  0001 C CNN
+F 1 "+9V" H 1200 2340 50  0000 C CNN
+F 2 "" H 1200 2200 50  0001 C CNN
+F 3 "" H 1200 2200 50  0001 C CNN
+	1    1200 2200
 	1    0    0    -1
 $EndComp
 Wire Wire Line
 	2250 3775 1825 3775
+$Comp
+L R R5
+U 1 1 59E60FCF
+P 1400 2475
+F 0 "R5" V 1480 2475 50  0000 C CNN
+F 1 "R" V 1400 2475 50  0000 C CNN
+F 2 "Resistors_SMD:R_0603" V 1330 2475 50  0001 C CNN
+F 3 "" H 1400 2475 50  0001 C CNN
+	1    1400 2475
+	1    0    0    -1
+$EndComp
+$Comp
+L Q_NPN_BCE Q3
+U 1 1 59E61059
+P 1725 2900
+F 0 "Q3" H 1925 2950 50  0000 L CNN
+F 1 "Q_NPN_BCE" H 1925 2850 50  0000 L CNN
+F 2 "TO_SOT_Packages_SMD:SOT-23" H 1925 3000 50  0001 C CNN
+F 3 "" H 1725 2900 50  0001 C CNN
+	1    1725 2900
+	1    0    0    -1
+$EndComp
+Wire Wire Line
+	1200 2200 1625 2200
+Wire Wire Line
+	1400 2325 1400 2200
+Connection ~ 1400 2200
+Wire Wire Line
+	1400 2625 1400 2700
+Wire Wire Line
+	1400 2700 1825 2700
+Wire Wire Line
+	1825 2700 1825 2500
+$Comp
+L R R4
+U 1 1 59E6131F
+P 1375 2900
+F 0 "R4" V 1455 2900 50  0000 C CNN
+F 1 "R" V 1375 2900 50  0000 C CNN
+F 2 "Resistors_SMD:R_0603" V 1305 2900 50  0001 C CNN
+F 3 "" H 1375 2900 50  0001 C CNN
+	1    1375 2900
+	0    1    1    0
+$EndComp
+Text Label 1225 2900 2    60   ~ 0
+PWREN
+$Comp
+L GND #PWR015
+U 1 1 59E613BB
+P 1825 3100
+F 0 "#PWR015" H 1825 2850 50  0001 C CNN
+F 1 "GND" H 1825 2950 50  0000 C CNN
+F 2 "" H 1825 3100 50  0001 C CNN
+F 3 "" H 1825 3100 50  0001 C CNN
+	1    1825 3100
+	1    0    0    -1
+$EndComp
+$Comp
+L Q_PMOS_GDS Q4
+U 1 1 59E61F36
+P 1825 2300
+F 0 "Q4" H 2025 2350 50  0000 L CNN
+F 1 "Q_PMOS_GDS" H 2025 2250 50  0000 L CNN
+F 2 "nixie-tube-fp:TO-252-2-ds" H 2025 2400 50  0001 C CNN
+F 3 "" H 1825 2300 50  0001 C CNN
+	1    1825 2300
+	0    1    -1   0
+$EndComp
 $EndSCHEMATC

Commit message: added and widen tracks of gnd and HV
Parts:
- C4: footprint Capacitors_SMD:C_0603 -> Capacitors_THT:CP_Radial_D8.0mm_P2.50mm
Changed lines of the file:
@@
 F 0 "C4" H 5975 3050 50  0000 L CNN
 F 1 "2.2uF" H 6000 2750 50  0000 L CNN
-F 2 "Capacitors_SMD:C_0603" H 5988 2800 50  0001 C CNN
+F 2 "Capacitors_THT:CP_Radial_D8.0mm_P2.50mm" H 5988 2800 50  0001 C CNN
 F 3 "" H 5950 2950 50  0000 C CNN
 F 4 "250V" H 6100 2850 60  0000 C CNN "voltage"

Commit message: fixed pin headers placement
Parts:
- removed J1: Conn_01x05_Male, Pin_Headers:Pin_Header_Angled_1x05_Pitch2.54mm, symbol Conn_01x05_Male
- removed J2: Conn_01x05_Female, Socket_Strips:Socket_Strip_Angled_1x05_Pitch2.54mm, symbol Conn_01x05_Female
- added J1: Conn_01x06_Male, Pin_Headers:Pin_Header_Angled_1x06_Pitch2.54mm, symbol Conn_01x06_Male
- added J2: Conn_01x06_Female, Socket_Strips:Socket_Strip_Angled_1x06_Pitch2.54mm, symbol Conn_01x06_Female
Connections:
- net +9V: now also J1.2 (Pin_2), J2.2 (Pin_2)
- net GND: now also J1.4 (Pin_4), J2.4 (Pin_4)
- net MOSi: now also J1.6 (Pin_6), J2.6 (Pin_6)
- net PWREN: now also J1.3 (Pin_3), J2.3 (Pin_3)
- net SCK: now also J1.5 (Pin_5), J2.5 (Pin_5)
- new net OE: J1.1 (Pin_1), J2.1 (Pin_1)
Changed lines of the file:
@@
 $EndComp
 $Comp
-L GND #PWR01
+L GND #PWR10
 U 1 1 59D51181
 P 4150 2600
-F 0 "#PWR01" H 4150 2350 50  0001 C CNN
+F 0 "#PWR10" H 4150 2350 50  0001 C CNN
 F 1 "GND" H 4150 2450 50  0000 C CNN
 F 2 "" H 4150 2600 50  0000 C CNN
@@
 $EndComp
 $Comp
-L GND #PWR02
+L GND #PWR14
 U 1 1 59D51419
 P 5550 4050
-F 0 "#PWR02" H 5550 3800 50  0001 C CNN
+F 0 "#PWR14" H 5550 3800 50  0001 C CNN
 F 1 "GND" H 5550 3900 50  0000 C CNN
 F 2 "" H 5550 4050 50  0000 C CNN
@@
 $EndComp
 $Comp
-L GND #PWR03
+L GND #PWR8
 U 1 1 59D51803
 P 3450 3500
-F 0 "#PWR03" H 3450 3250 50  0001 C CNN
+F 0 "#PWR8" H 3450 3250 50  0001 C CNN
 F 1 "GND" H 3450 3350 50  0000 C CNN
 F 2 "" H 3450 3500 50  0000 C CNN
@@
 $EndComp
 $Comp
-L GND #PWR04
+L GND #PWR12
 U 1 1 59D51D24
 P 4800 3300
-F 0 "#PWR04" H 4800 3050 50  0001 C CNN
+F 0 "#PWR12" H 4800 3050 50  0001 C CNN
 F 1 "GND" H 4800 3150 50  0000 C CNN
 F 2 "" H 4800 3300 50  0000 C CNN
@@
 PULSE OUT
 $Comp
-L GND #PWR05
+L GND #PWR13
 U 1 1 59D522B9
 P 5300 4050
-F 0 "#PWR05" H 5300 3800 50  0001 C CNN
+F 0 "#PWR13" H 5300 3800 50  0001 C CNN
 F 1 "GND" H 5300 3900 50  0000 C CNN
 F 2 "" H 5300 4050 50  0000 C CNN
@@
 $EndComp
 $Comp
-L GND #PWR06
+L GND #PWR15
 U 1 1 59D524CC
 P 5950 3300
-F 0 "#PWR06" H 5950 3050 50  0001 C CNN
+F 0 "#PWR15" H 5950 3050 50  0001 C CNN
 F 1 "GND" H 5950 3150 50  0000 C CNN
 F 2 "" H 5950 3300 50  0000 C CNN
@@
 1.25V
 $Comp
-L GND #PWR07
+L GND #PWR7
 U 1 1 59D52828
 P 3050 3600
-F 0 "#PWR07" H 3050 3350 50  0001 C CNN
+F 0 "#PWR7" H 3050 3350 50  0001 C CNN
 F 1 "GND" H 3050 3450 50  0000 C CNN
 F 2 "" H 3050 3600 50  0000 C CNN
@@
 +180V
 $Comp
-L GND #PWR08
+L GND #PWR9
 U 1 1 59D52C94
 P 3950 3700
-F 0 "#PWR08" H 3950 3450 50  0001 C CNN
+F 0 "#PWR9" H 3950 3450 50  0001 C CNN
 F 1 "GND" H 3950 3550 50  0000 C CNN
 F 2 "" H 3950 3700 50  0000 C CNN
@@
 $EndComp
 $Comp
-L GND #PWR09
+L GND #PWR11
 U 1 1 59D52CCD
 P 4300 3700
-F 0 "#PWR09" H 4300 3450 50  0001 C CNN
+F 0 "#PWR11" H 4300 3450 50  0001 C CNN
 F 1 "GND" H 4300 3550 50  0000 C CNN
 F 2 "" H 4300 3700 50  0000 C CNN
@@
 $EndComp
 $Comp
-L GND #PWR010
+L GND #PWR4
 U 1 1 59D51046
 P 2450 3925
-F 0 "#PWR010" H 2450 3675 50  0001 C CNN
+F 0 "#PWR4" H 2450 3675 50  0001 C CNN
 F 1 "GND" H 2450 3775 50  0000 C CNN
 F 2 "" H 2450 3925 50  0000 C CNN
@@
 F 3 "" H 6550 2325 50  0001 C CNN
 	1    6550 2325
-	1    0    0    -1
-$EndComp
-$Comp
-L Conn_01x05_Female J2
-U 1 1 59E5DA12
-P 3275 4900
-F 0 "J2" H 3275 5200 50  0000 C CNN
-F 1 "Conn_01x05_Female" H 3275 4600 50  0000 C CNN
-F 2 "Socket_Strips:Socket_Strip_Angled_1x05_Pitch2.54mm" H 3275 4900 50  0001 C CNN
-F 3 "" H 3275 4900 50  0001 C CNN
-	1    3275 4900
-	1    0    0    -1
-$EndComp
-$Comp
-L Conn_01x05_Male J1
-U 1 1 59E5DABD
-P 2000 4900
-F 0 "J1" H 2000 5200 50  0000 C CNN
-F 1 "Conn_01x05_Male" H 2000 4600 50  0000 C CNN
-F 2 "Pin_Headers:Pin_Header_Angled_1x05_Pitch2.54mm" H 2000 4900 50  0001 C CNN
-F 3 "" H 2000 4900 50  0001 C CNN
-	1    2000 4900
 	1    0    0    -1
 $EndComp
@@
 MOSi
 $Comp
-L +9V #PWR011
+L +9V #PWR3
 U 1 1 59E5E8EF
 P 2250 3700
-F 0 "#PWR011" H 2250 3550 50  0001 C CNN
+F 0 "#PWR3" H 2250 3550 50  0001 C CNN
 F 1 "+9V" H 2250 3840 50  0000 C CNN
 F 2 "" H 2250 3700 50  0001 C CNN
@@
 	2250 3775 2250 3700
 $Comp
-L +9V #PWR012
+L +9V #PWR5
 U 1 1 59E5EF02
 P 2675 4500
-F 0 "#PWR012" H 2675 4350 50  0001 C CNN
+F 0 "#PWR5" H 2675 4350 50  0001 C CNN
 F 1 "+9V" H 2675 4640 50  0000 C CNN
 F 2 "" H 2675 4500 50  0001 C CNN
@@
 Connection ~ 2675 4700
 $Comp
-L GND #PWR013
+L GND #PWR6
 U 1 1 59E5EFC2
 P 2900 4600
-F 0 "#PWR013" H 2900 4350 50  0001 C CNN
+F 0 "#PWR6" H 2900 4350 50  0001 C CNN
 F 1 "GND" H 2900 4450 50  0000 C CNN
 F 2 "" H 2900 4600 50  0001 C CNN
@@
 	2025 2200 4800 2200
 $Comp
-L +9V #PWR014
+L +9V #PWR1
 U 1 1 59E606F5
 P 1200 2200
-F 0 "#PWR014" H 1200 2050 50  0001 C CNN
+F 0 "#PWR1" H 1200 2050 50  0001 C CNN
 F 1 "+9V" H 1200 2340 50  0000 C CNN
 F 2 "" H 1200 2200 50  0001 C CNN
@@
 PWREN
 $Comp
-L GND #PWR015
+L GND #PWR2
 U 1 1 59E613BB
 P 1825 3100
-F 0 "#PWR015" H 1825 2850 50  0001 C CNN
+F 0 "#PWR2" H 1825 2850 50  0001 C CNN
 F 1 "GND" H 1825 2950 50  0000 C CNN
 F 2 "" H 1825 3100 50  0001 C CNN
@@
 	0    1    -1   0
 $EndComp
+$Comp
+L Conn_01x06_Male J1
+U 1 1 59F6FE01
+P 2000 4800
+F 0 "J1" H 2000 5100 50  0000 C CNN
+F 1 "Conn_01x06_Male" H 2000 4400 50  0000 C CNN
+F 2 "Pin_Headers:Pin_Header_Angled_1x06_Pitch2.54mm" H 2000 4800 50  0001 C CNN
+F 3 "" H 2000 4800 50  0001 C CNN
+	1    2000 4800
+	1    0    0    -1
+$EndComp
+$Comp
+L Conn_01x06_Female J2
+U 1 1 59F70E4E
+P 3275 4800
+F 0 "J2" H 3275 5100 50  0000 C CNN
+F 1 "Conn_01x06_Female" H 3275 4400 50  0000 C CNN
+F 2 "Socket_Strips:Socket_Strip_Angled_1x06_Pitch2.54mm" H 3275 4800 50  0001 C CNN
+F 3 "" H 3275 4800 50  0001 C CNN
+	1    3275 4800
+	1    0    0    -1
+$EndComp
+Wire Wire Line
+	2200 4600 3075 4600
+Text Label 2200 4600 0    60   ~ 0
+OE
 $EndSCHEMATC

Commit message: finalize layout
Parts:
- Q4: value Q_PMOS_GDS -> AO3400; footprint nixie-tube-fp:TO-252-2-ds -> TO_SOT_Packages_SMD:SOT-23
Changed lines of the file:
@@
 $EndComp
 $Comp
-L GND #PWR10
+L GND #PWR01
 U 1 1 59D51181
 P 4150 2600
-F 0 "#PWR10" H 4150 2350 50  0001 C CNN
+F 0 "#PWR01" H 4150 2350 50  0001 C CNN
 F 1 "GND" H 4150 2450 50  0000 C CNN
 F 2 "" H 4150 2600 50  0000 C CNN
@@
 $EndComp
 $Comp
-L GND #PWR14
+L GND #PWR02
 U 1 1 59D51419
 P 5550 4050
-F 0 "#PWR14" H 5550 3800 50  0001 C CNN
+F 0 "#PWR02" H 5550 3800 50  0001 C CNN
 F 1 "GND" H 5550 3900 50  0000 C CNN
 F 2 "" H 5550 4050 50  0000 C CNN
@@
 $EndComp
 $Comp
-L GND #PWR8
+L GND #PWR03
 U 1 1 59D51803
 P 3450 3500
-F 0 "#PWR8" H 3450 3250 50  0001 C CNN
+F 0 "#PWR03" H 3450 3250 50  0001 C CNN
 F 1 "GND" H 3450 3350 50  0000 C CNN
 F 2 "" H 3450 3500 50  0000 C CNN
@@
 $EndComp
 $Comp
-L GND #PWR12
+L GND #PWR04
 U 1 1 59D51D24
 P 4800 3300
-F 0 "#PWR12" H 4800 3050 50  0001 C CNN
+F 0 "#PWR04" H 4800 3050 50  0001 C CNN
 F 1 "GND" H 4800 3150 50  0000 C CNN
 F 2 "" H 4800 3300 50  0000 C CNN
@@
 PULSE OUT
 $Comp
-L GND #PWR13
+L GND #PWR05
 U 1 1 59D522B9
 P 5300 4050
-F 0 "#PWR13" H 5300 3800 50  0001 C CNN
+F 0 "#PWR05" H 5300 3800 50  0001 C CNN
 F 1 "GND" H 5300 3900 50  0000 C CNN
 F 2 "" H 5300 4050 50  0000 C CNN
@@
 $EndComp
 $Comp
-L GND #PWR15
+L GND #PWR06
 U 1 1 59D524CC
 P 5950 3300
-F 0 "#PWR15" H 5950 3050 50  0001 C CNN
+F 0 "#PWR06" H 5950 3050 50  0001 C CNN
 F 1 "GND" H 5950 3150 50  0000 C CNN
 F 2 "" H 5950 3300 50  0000 C CNN
@@
 1.25V
 $Comp
-L GND #PWR7
+L GND #PWR07
 U 1 1 59D52828
 P 3050 3600
-F 0 "#PWR7" H 3050 3350 50  0001 C CNN
+F 0 "#PWR07" H 3050 3350 50  0001 C CNN
 F 1 "GND" H 3050 3450 50  0000 C CNN
 F 2 "" H 3050 3600 50  0000 C CNN
@@
 +180V
 $Comp
-L GND #PWR9
+L GND #PWR08
 U 1 1 59D52C94
 P 3950 3700
-F 0 "#PWR9" H 3950 3450 50  0001 C CNN
+F 0 "#PWR08" H 3950 3450 50  0001 C CNN
 F 1 "GND" H 3950 3550 50  0000 C CNN
 F 2 "" H 3950 3700 50  0000 C CNN
@@
 $EndComp
 $Comp
-L GND #PWR11
+L GND #PWR09
 U 1 1 59D52CCD
 P 4300 3700
-F 0 "#PWR11" H 4300 3450 50  0001 C CNN
+F 0 "#PWR09" H 4300 3450 50  0001 C CNN
 F 1 "GND" H 4300 3550 50  0000 C CNN
 F 2 "" H 4300 3700 50  0000 C CNN
@@
 $EndComp
 $Comp
-L GND #PWR4
+L GND #PWR010
 U 1 1 59D51046
 P 2450 3925
-F 0 "#PWR4" H 2450 3675 50  0001 C CNN
+F 0 "#PWR010" H 2450 3675 50  0001 C CNN
 F 1 "GND" H 2450 3775 50  0000 C CNN
 F 2 "" H 2450 3925 50  0000 C CNN
@@
 MOSi
 $Comp
-L +9V #PWR3
+L +9V #PWR011
 U 1 1 59E5E8EF
 P 2250 3700
-F 0 "#PWR3" H 2250 3550 50  0001 C CNN
+F 0 "#PWR011" H 2250 3550 50  0001 C CNN
 F 1 "+9V" H 2250 3840 50  0000 C CNN
 F 2 "" H 2250 3700 50  0001 C CNN
@@
 	2250 3775 2250 3700
 $Comp
-L +9V #PWR5
+L +9V #PWR012
 U 1 1 59E5EF02
 P 2675 4500
-F 0 "#PWR5" H 2675 4350 50  0001 C CNN
+F 0 "#PWR012" H 2675 4350 50  0001 C CNN
 F 1 "+9V" H 2675 4640 50  0000 C CNN
 F 2 "" H 2675 4500 50  0001 C CNN
@@
 Connection ~ 2675 4700
 $Comp
-L GND #PWR6
+L GND #PWR013
 U 1 1 59E5EFC2
 P 2900 4600
-F 0 "#PWR6" H 2900 4350 50  0001 C CNN
+F 0 "#PWR013" H 2900 4350 50  0001 C CNN
 F 1 "GND" H 2900 4450 50  0000 C CNN
 F 2 "" H 2900 4600 50  0001 C CNN
@@
 	2025 2200 4800 2200
 $Comp
-L +9V #PWR1
+L +9V #PWR014
 U 1 1 59E606F5
 P 1200 2200
-F 0 "#PWR1" H 1200 2050 50  0001 C CNN
+F 0 "#PWR014" H 1200 2050 50  0001 C CNN
 F 1 "+9V" H 1200 2340 50  0000 C CNN
 F 2 "" H 1200 2200 50  0001 C CNN
@@
 PWREN
 $Comp
-L GND #PWR2
+L GND #PWR015
 U 1 1 59E613BB
 P 1825 3100
-F 0 "#PWR2" H 1825 2850 50  0001 C CNN
+F 0 "#PWR015" H 1825 2850 50  0001 C CNN
 F 1 "GND" H 1825 2950 50  0000 C CNN
 F 2 "" H 1825 3100 50  0001 C CNN
@@
 P 1825 2300
 F 0 "Q4" H 2025 2350 50  0000 L CNN
-F 1 "Q_PMOS_GDS" H 2025 2250 50  0000 L CNN
-F 2 "nixie-tube-fp:TO-252-2-ds" H 2025 2400 50  0001 C CNN
+F 1 "AO3400" H 2025 2250 50  0000 L CNN
+F 2 "TO_SOT_Packages_SMD:SOT-23" H 2025 2400 50  0001 C CNN
 F 3 "" H 1825 2300 50  0001 C CNN
 	1    1825 2300

Commit message: fixed pin position not in sequence with other board
Connections:
- net +9V: now also J1.5 (Pin_5), J2.5 (Pin_5); no longer J1.2 (Pin_2), J2.2 (Pin_2)
- net GND: now also J1.3 (Pin_3), J2.3 (Pin_3); no longer J1.4 (Pin_4), J2.4 (Pin_4)
- net MOSi: now also J1.1 (Pin_1), J2.1 (Pin_1); no longer J1.6 (Pin_6), J2.6 (Pin_6)
- net OE: now also J1.6 (Pin_6), J2.6 (Pin_6); no longer J1.1 (Pin_1), J2.1 (Pin_1)
- net PWREN: now also J1.4 (Pin_4), J2.4 (Pin_4); no longer J1.3 (Pin_3), J2.3 (Pin_3)
- net SCK: now also J1.2 (Pin_2), J2.2 (Pin_2); no longer J1.5 (Pin_5), J2.5 (Pin_5)
Changed lines of the file:
@@
 L Conn_01x06_Male J1
 U 1 1 59F6FE01
-P 2000 4800
-F 0 "J1" H 2000 5100 50  0000 C CNN
-F 1 "Conn_01x06_Male" H 2000 4400 50  0000 C CNN
-F 2 "Pin_Headers:Pin_Header_Angled_1x06_Pitch2.54mm" H 2000 4800 50  0001 C CNN
-F 3 "" H 2000 4800 50  0001 C CNN
-	1    2000 4800
-	1    0    0    -1
+P 2000 4900
+F 0 "J1" H 2000 5200 50  0000 C CNN
+F 1 "Conn_01x06_Male" H 2000 4500 50  0000 C CNN
+F 2 "Pin_Headers:Pin_Header_Angled_1x06_Pitch2.54mm" H 2000 4900 50  0001 C CNN
+F 3 "" H 2000 4900 50  0001 C CNN
+	1    2000 4900
+	1    0    0    1
 $EndComp
 $Comp
 L Conn_01x06_Female J2
 U 1 1 59F70E4E
-P 3275 4800
-F 0 "J2" H 3275 5100 50  0000 C CNN
-F 1 "Conn_01x06_Female" H 3275 4400 50  0000 C CNN
-F 2 "Socket_Strips:Socket_Strip_Angled_1x06_Pitch2.54mm" H 3275 4800 50  0001 C CNN
-F 3 "" H 3275 4800 50  0001 C CNN
-	1    3275 4800
-	1    0    0    -1
+P 3275 4900
+F 0 "J2" H 3275 5200 50  0000 C CNN
+F 1 "Conn_01x06_Female" H 3275 4500 50  0000 C CNN
+F 2 "Socket_Strips:Socket_Strip_Angled_1x06_Pitch2.54mm" H 3275 4900 50  0001 C CNN
+F 3 "" H 3275 4900 50  0001 C CNN
+	1    3275 4900
+	1    0    0    1
 $EndComp
 Wire Wire Line
