File: nixie_tube.kicad_pcb (KiCad board)
At the start: 2 copper layers, 25 x 44 mm, 14 parts, among them P1 CONN_01X02, Q1 MPSA92, Q2 IRF740, U1 MC34063

Commit message: finalize position of component
Parts:
- removed P1: CONN_01X02, Pin_Headers:Pin_Header_Angled_1x02
- added J1: Conn_01x05_Male, Pin_Headers:Pin_Header_Angled_1x05_Pitch2.54mm, F.Cu at (178.0, 125.5)
- added J11: dc003a, nixie-tube-fp:dc005a, F.Cu at (187.0, 125.5)
- added J2: Conn_01x05_Female, Socket_Strips:Socket_Strip_Angled_1x05_Pitch2.54mm, F.Cu at (191.5, 125.5)
- added J3: Conn_01x01_Male, Pin_Headers:Pin_Header_Angled_1x01_Pitch2.54mm, F.Cu at (178.0, 86.5)
- added J4: Conn_01x01_Female, Socket_Strips:Socket_Strip_Angled_1x01_Pitch2.54mm, F.Cu at (191.5, 86.0)
- added Q3: Q_NPN_BCE, TO_SOT_Packages_SMD:SOT-23, F.Cu at (169.5, 110.5)
- added Q4: Q_PMOS_GDS, nixie-tube-fp:TO-252-2-ds, F.Cu at (171.2, 101.1)
- added R4: R, Resistors_SMD:R_0603, F.Cu at (177.5, 104.5)
- added R5: R, Resistors_SMD:R_0603, F.Cu at (177.5, 102.5)
- C1: value CP -> 20nF; footprint Capacitors_SMD:C_0603_HandSoldering -> Capacitors_SMD:C_0603
- C2: footprint Capacitors_SMD:C_0603_HandSoldering -> nixie-tube-fp:220uF-35V-smd
- C3, C4: footprint Capacitors_SMD:C_0603_HandSoldering -> Capacitors_SMD:C_0603
- D1: value 1N914 -> 1N4148; footprint Diodes_SMD:DO-214AB_Handsoldering -> Diodes_SMD:D_SOD-123
- D2: value BAV21 -> RS2M; footprint Diodes_SMD:DO-214AB_Handsoldering -> Diodes_SMD:D_SMA
- Q1: value MPSA92 -> SS8550
- Q2: value IRF740 -> FQD5N60C
- R1: footprint Resistors_SMD:R_0603_HandSoldering -> Resistors_SMD:R_0603
- R2: value 475K -> 470K; footprint Resistors_SMD:R_0603_HandSoldering -> Resistors_SMD:R_0603
- R3: value 3K32 -> 3K; footprint Resistors_SMD:R_0603_HandSoldering -> Resistors_SMD:R_0603
- moved R3 24.0 mm to (190.0, 111.5), turned to 0 degrees
- moved C4 22.2 mm to (190.0, 105.5), turned to 0 degrees
- moved R2 21.6 mm to (190.0, 109.5)
- moved C3 20.1 mm to (190.0, 107.5), turned to 0 degrees
- moved C2 18.4 mm to (189.0, 92.5)
- moved D1 16.1 mm to (176.5, 110.0)
- moved C1 11.2 mm to (183.0, 100.5), turned to 270 degrees
- moved Q2 10.6 mm to (184.0, 113.3)
- moved U1 9.85 mm to (189.0, 100.5)
- moved L1 9.51 mm to (171.5, 92.5), turned to 0 degrees
- moved R1 9.22 mm to (181.0, 100.5), turned to 270 degrees
- moved Q1 8.32 mm to (177.5, 98.5), turned to 270 degrees
- moved D2 6.08 mm to (180.5, 92.0), turned to 0 degrees
Routing:
- net (no net): vias 1 -> 0
Other:
- board size 25 x 44 mm -> 28 x 44 mm

Commit message: rearrange components
Parts:
- moved C1 11.1 mm to (184.5, 111.5)
- moved R1 11.1 mm to (182.5, 111.5)
- moved Q2 10.6 mm to (180.0, 103.5)
- moved Q1 9.01 mm to (180.5, 107.0)
- moved R4 7.76 mm to (175.5, 112.0)
- moved R5 7.76 mm to (175.5, 110.0)
- moved D1 3.35 mm to (179.5, 111.5)
- moved J4 0.50 mm to (191.5, 86.5)
- turned C3 to 180 degrees
- turned R2 to 0 degrees
- turned R3 to 180 degrees
Routing:
- net Net-(C4-Pad1): track 0.00 -> 47.9 mm
- net GND: track 0.00 -> 30.3 mm
- net /PWREN: track 0.00 -> 25.2 mm
- net +9V: track 0.00 -> 22.4 mm
- net Net-(D1-Pad2): track 0.00 -> 21.1 mm
- net Net-(C2-Pad1): track 0.00 -> 19.0 mm
- net Net-(D2-Pad2): track 0.00 -> 16.7 mm
- net /SCK: track 0.00 -> 13.5 mm
- net /MOSi: track 0.00 -> 13.5 mm
- net Net-(C1-Pad1): track 0.00 -> 11.6 mm
- net Net-(Q3-Pad2): track 0.00 -> 11.4 mm
- net Net-(C3-Pad1): track 0.00 -> 9.50 mm
- net Net-(D1-Pad1): track 0.00 -> 8.26 mm
- net Net-(Q3-Pad1): track 0.00 -> 5.34 mm
Other:
- net class 9V added: clearance 0.2, trace_width 0.5, via_dia 0.6, via_drill 0.4
- net class GND added: clearance 0.2, trace_width 0.4, via_dia 0.6, via_drill 0.4

Commit message: finished routed
Parts:
- moved C2 1.00 mm to (189.0, 93.5)
Routing:
- net GND: track 30.3 -> 52.1 mm, vias 0 -> 7
- net Net-(C2-Pad1): track 19.0 -> 33.7 mm
- net Net-(C4-Pad1): track 47.9 -> 61.9 mm
- net +9V: track 22.4 -> 32.9 mm, vias 0 -> 2
- net /SCK: track 13.5 -> 14.2 mm
- added copper zone on F.Cu, net +9V
- added copper zone on B.Cu, net GND
Other:
- board text added: "28x44mm"
